File: board1.sch (EAGLE design)
At the start: 0 parts

Commit message: Copied the last schematic from demo PCB
Parts:
- added ADC: ADS1256IDBT, SSOP_Breakout_Boards_SdR:ADS1256IDBT
- added AIN6-7: (no value), SparkFun-Connectors:M02PTH
- added BEAGLE_POW, JP1A, JP1B, JP2A, JP2B: (no value), SparkFun-Connectors:M03PTH
- added C1, C6: 10u, adafruit:C-USC3216
- added C10, C12, C14, C16, C17, C2, C4, C7: 0.1u, adafruit:C-USC3216
- added C11, C13, C15, C5: 100p, adafruit:C-USC3216
- added C18: 1u, adafruit:C-USC3216
- added C3: 47u, adafruit:C-USC3216
- added C8, C9: 18p, adafruit:C-USC3216
- added DIG_OUT, RESET/SYNC: (no value), SparkFun-Connectors:M04PTH
- added F1: 15A, fuse:SHK20L
- added Q1: 7.68M, adafruit:CRYSTALHC49U-V
- added R1: 0.005, LVK25:LVK25R001
- added R2A40, R2B40: 560k, adafruit:R-US_M3216
- added R2A400, R2B400: 5.49M, adafruit:R-US_M3216
- added R3A, R3B: 1k, adafruit:R-US_M3216
- added R4, R5: 49.9, adafruit:R-US_R2512
- added R6, R7, R8: 100, adafruit:R-US_M3216
- added SERIAL: (no value), SparkFun-Connectors:M05PTH
- added VBOX, VPANEL: 2PIN_TERMINAL_PCBMOUNT, TE CONNECTIVITY:2PIN_TERMINAL_PCBMOUNT
- added VOLTAGE_REF: ADR3425ARJZ-R7, Analog Devices_By_element14_Batch_1:ADR3425ARJZ-R7
Connections:
- new net AIN0: ADC.AIN0, C10.2, C11.2, R1.2
- new net AIN1: ADC.AIN1, C10.1, C11.1, R1.4
- new net AIN2: ADC.AIN2, C12.1, C13.1, JP2B.2, R3B.2
- new net AIN3: ADC.AIN3, C12.2, C13.2, R1.3, R3B.1, VBOX.2
- new net AIN4: ADC.AIN4, C14.1, C15.1, JP2A.2, R3A.2
- new net AIN5: ADC.AIN5, C14.2, C15.2, F1.2A, F1.2B, R1.1, R3A.1
- new net BEAGLE_3V3: ADC.DVDD, BEAGLE_POW.1, C6.1, C7.1
- new net BEAGLE_5V: ADC.AVDD, BEAGLE_POW.3, C1.1, C17.1, C18.1, C2.1, VOLTAGE_REF.EN, VOLTAGE_REF.VIN
- new net BEAGLE_GND: ADC.AGND, ADC.AINCOM, ADC.DGND, BEAGLE_POW.2, C1.2, C16.2, C17.2, C18.2, C2.2, C6.2, C7.2, C8.2, C9.2, R4.1, RESET/SYNC.2, RESET/SYNC.3, VOLTAGE_REF.GND_FORCE
- new net D0: ADC.D0/CLKOUT, DIG_OUT.1
- new net DIN: ADC.DIN, R7.2
- new net DOUT: ADC.DOUT, SERIAL.3
- new net N$10: JP2B.1, R2B40.1
- new net N$11: ADC.XTAL1/CLKIN, C8.1, Q1.1
- new net N$12: ADC.XTAL2, C9.1, Q1.2
- new net N$13: ADC.D2, DIG_OUT.3
- new net N$15: ADC.D3, DIG_OUT.4
- new net N$16: R7.1, SERIAL.2
- new net N$17: R6.1, SERIAL.1
- new net N$18: ADC.AIN6, AIN6-7.2
- new net N$19: ADC.AIN7, AIN6-7.1
- new net N$2: JP1A.3, R2A40.2
- new net N$22: R8.1, SERIAL.5
- new net N$23: C16.1, R5.1, VOLTAGE_REF.VOUT_FORCE
- new net N$3: JP1A.1, R2A400.2
- new net N$4: JP2A.3, R2A400.1
- new net N$5: JP2A.1, R2A40.1
- new net N$6: ADC.D1, DIG_OUT.2
- new net N$7: JP1B.3, R2B40.2
- new net N$8: JP1B.1, R2B400.2
- new net N$9: JP2B.3, R2B400.1
- new net SCLK: ADC.SCLK, R6.2
- new net VBUS1: JP1A.2, JP1B.2, VBOX.1, VPANEL.1
- new net VBUS2: F1.1A, F1.1B, VPANEL.2
- new net VREFN: ADC.VREFN, C3.2, C4.2, C5.2, R4.2, VOLTAGE_REF.GND_SEN
- new net VREFP: ADC.VREFP, C3.1, C4.1, C5.1, R5.2, VOLTAGE_REF.VOUT_SEN
- new net ~CS: ADC.~CS, R8.2
- new net ~DRDY: ADC.~DRDY, SERIAL.4
- new net ~RESET: ADC.~RESET, RESET/SYNC.4
- new net ~SYNC: ADC.~SYNC,_~PDWN, RESET/SYNC.1
