File: board1.sch (EAGLE design)
At the start: 44 parts, among them Q1 7.68M, U1 ADS1256IDBT

Commit message: Added atmega, RTC, ICSP header, Resert button. Organized the schematic with borders
Parts:
- removed C18: 1u, adafruit:C-USC3216
- added ATMEGA328: ATMEGA328P_TQFP, SparkFun-DigitalIC:ATMEGA328P_TQFP
- added DC-DC: ADUM5000ARWZ, Analog Devices_By_element14_Batch_1:ADUM5000ARWZ
- added IC1: IC_DIL16-SOIC-16, MAX14850ASE:IC_DIL16-SOIC-16
- added ICSP: FEMALE 2x3, SparkFun-Connectors:M03X2FEMALE
- added RESET_BUTTON: TAC_SWITCHSMD, SparkFun-Retired:TAC_SWITCHSMD
- added RTC: DS3234, SparkFun-FreqCtrl:DS3234
Connections:
- net BEAGLE_5V: no longer C18.1
- net BEAGLE_GND: no longer C18.2
Other:
- note added: "Connectors"
- note added: "DS1256 ADC"
- note added: "Electrical Measurements"
- note added: "Isolation"
- note added: "March 2016"
- note added: "Measuring PCB"
- note added: "Real Time Clock"
- note added: "Sideridis Paschalis"
- note added: "Standalone Arduino (atmega328)"
- note added: "This board measures Voltage, Current and Temperature. In addition, it get a Date and Time stamp. The data are collected from the microprocessor Atmega328 and send out as I2C packages. Isolation is placed in every connection outside the board"
- note added: "Voltage Reference for ADC"
- note added: "date"
- note added: "description"
- note added: "designer"
- note added: "title"
- moved on the sheet: AIN6-7, BEAGLE_POW, C1, C10, C11, C12, C13, C14, C15, C16, C17, C2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

Commit message: Added connectors, 3v3 regulator. Almost finished the schematic.
Parts:
- removed BEAGLE_POW: (no value), SparkFun-Connectors:M03PTH
- removed DIG_OUT: (no value), SparkFun-Connectors:M04PTH
- removed IC1: IC_DIL16-SOIC-16, MAX14850ASE:IC_DIL16-SOIC-16
- removed SERIAL: (no value), SparkFun-Connectors:M05PTH
- removed U1: ADS1256IDBT, Texas Instruments_By_element14_Batch_1:ADS1256IDBT
- removed VOLTAGE_REF: ADR3425ARJZ-R7, Analog Devices_By_element14_Batch_1:ADR3425ARJZ-R7
- added 2V5_VOLTAGE_REF: ADR3425ARJZ-R7, Analog Devices_By_element14_Batch_1:ADR3425ARJZ-R7
- added 3V3_REGULATOR: LP2985-33DBVT, Texas Instruments_By_element14_Batch_1:LP2985-33DBVT
- added ADC: ADS1256IDBT, Texas Instruments_By_element14_Batch_1:ADS1256IDBT
- added C18, C20, C23, C25: 10u, SparkFun-Capacitors:CAP1206
- added C19, C21, C22, C24, C26, C27: 0.1u, SparkFun-Capacitors:CAP1206
- added C28: 1u, SparkFun-Capacitors:CAP1206
- added C29: 10n, SparkFun-Capacitors:CAP1206
- added C30: 2.2u, SparkFun-Capacitors:CAP1206
- added C31, C32, C33, C34: 22p, SparkFun-Capacitors:CAP1206
- added Q2: 16MHz, adafruit:CRYSTALHC49U-V
- added R10, R2, R3, R4, R5: 4.7k, SparkFun-Passives:RESISTOR1206
- added R11, R9: 10k, SparkFun-Passives:RESISTOR1206
- added SIGNAL_ISOLATOR: IC_DIL16-SOIC-16, MAX14850ASE:IC_DIL16-SOIC-16
- added TO_MASTER_BOARD: (no value), pinhead:PINHD-1X8/90
Connections:
- removed net BEAGLE_3V3: BEAGLE_POW.1, C6.1, C7.1, SJ1.1, SJ2.1, U1.DVDD
- removed net BEAGLE_5V: BEAGLE_POW.3, C1.1, C17.1, C2.1, U1.AVDD, VOLTAGE_REF.EN, VOLTAGE_REF.VIN
- removed net BEAGLE_GND: BEAGLE_POW.2, C1.2, C16.2, C17.2, C2.2, C3.2, C4.2, C5.2, C6.2, C7.2, C8.2, C9.2, U1.AGND, U1.AINCOM, U1.DGND, U1.VREFN, VOLTAGE_REF.GND_FORCE, VOLTAGE_REF.GND_SEN
- removed net D0: DIG_OUT.1, U1.D0/CLKOUT
- removed net DIN: R7.2, U1.DIN
- removed net DOUT: SERIAL.3, U1.DOUT
- removed net N$15: DIG_OUT.4, U1.D3
- removed net N$22: R8.1, SERIAL.5
- removed net VREFP: C16.1, C3.1, C4.1, C5.1, U1.VREFP, VOLTAGE_REF.VOUT_FORCE, VOLTAGE_REF.VOUT_SEN
- removed net ~CS: R8.2, U1.~CS
- removed net ~DRDY: SERIAL.4, U1.~DRDY
- removed net ~RESET: SJ2.2, U1.~RESET
- removed net ~SYNC: SJ1.2, U1.~SYNC,_~PDWN
- new net 1WIRE_BUS: ATMEGA328.PD4(XCK/T0), R10.2
- new net 3V3: 3V3_REGULATOR.VOUT, ADC.DVDD, C30.1, C31.1, C6.1, C7.1, R9.2, RTC.VCC, SJ1.1, SJ2.1
- new net 5V: C18.1, C19.1, C20.1, C21.1, C26.1, DC-DC.RCSEL, DC-DC.VDD1, DC-DC.VDD1_2, ICSP.2, R2.2, R3.2, SIGNAL_ISOLATOR.VCCA, TO_MASTER_BOARD.1
- new net 5V_ISO: 2V5_VOLTAGE_REF.EN, 2V5_VOLTAGE_REF.VIN, 3V3_REGULATOR.ON/_~OFF, 3V3_REGULATOR.VIN, ADC.AVDD, ATMEGA328.AVCC, ATMEGA328.VCC@4, ATMEGA328.VCC@6, C1.1, C17.1, C2.1, C22.1, C23.1, C24.1, C25.1, C27.1, C27.2, C28.1, C34.2, DC-DC.VISO, DC-DC.VISO_2, DC-DC.VSEL, R10.1, R11.1, R4.2, R5.2, SIGNAL_ISOLATOR.GNDB, SIGNAL_ISOLATOR.VCCB
- new net ADC_CS: ATMEGA328.PD7(AIN1), R8.2
- new net ADC_DRDY: ADC.~DRDY, ATMEGA328.PD2(INT0)
- new net GND: C18.2, C19.2, C20.2, C21.2, C26.2, DC-DC.GND1, DC-DC.GND1_2, DC-DC.NC_2, ICSP.6, SIGNAL_ISOLATOR.GNDA, TO_MASTER_BOARD.2
- new net GND_ISO: 2V5_VOLTAGE_REF.GND_FORCE, 2V5_VOLTAGE_REF.GND_SEN, 3V3_REGULATOR.GND, ADC.AGND, ADC.AINCOM, ADC.DGND, ADC.VREFN, ATMEGA328.AGND, ATMEGA328.GND@3, ATMEGA328.GND@5, C1.2, C16.2, C17.2, C2.2, C22.2, C23.2, C24.2, C25.2, C28.2, C29.2, C3.2, C30.2, C31.2, C32.1, C33.1, C34.1, C4.2, C5.2, C6.2, C7.2, C8.2, C9.2, DC-DC.GNDISO, DC-DC.GNDISO_2, DC-DC.NC, RESET_BUTTON.1, RESET_BUTTON.2, RTC.GND, RTC.GND@10, RTC.GND@11, RTC.GND@12, RTC.GND@13, RTC.GND@14, RTC.GND@2, RTC.GND@7, RTC.GND@8, RTC.GND@9
- new net IN1: SIGNAL_ISOLATOR.INA1, TO_MASTER_BOARD.5
- new net IN2: SIGNAL_ISOLATOR.INA2, TO_MASTER_BOARD.6
- new net IN2_ISO: SIGNAL_ISOLATOR.OUTB2
- new net MISO: ADC.DOUT, ATMEGA328.PB4(MISO), ICSP.1, RTC.DOUT
- new net MOSI: ATMEGA328.PB3(MOSI/OC2), ICSP.4, R7.2, RTC.DIN
- new net N$1: ADC.SCLK, R6.1
- new net N$14: ADC.DIN, R7.1
- new net N$20: ADC.~SYNC,_~PDWN, SJ2.2
- new net N$21: 3V3_REGULATOR.BYPASS, C29.1
- new net OUT1: SIGNAL_ISOLATOR.OUTA1, TO_MASTER_BOARD.7
- new net OUT1_ISO: ATMEGA328.PD6(AIN0), SIGNAL_ISOLATOR.INB1
- new net OUT2: SIGNAL_ISOLATOR.OUTA2, TO_MASTER_BOARD.8
- new net OUT2_ISO: SIGNAL_ISOLATOR.INB2
- new net RESET: ATMEGA328.PC6(/RESET), ICSP.5, R11.2, RESET_BUTTON.3, RESET_BUTTON.4, SIGNAL_ISOLATOR.OUTB1
- new net RTC_CS: ATMEGA328.PB0(ICP), RTC.CS
- new net RTC_SQW: ATMEGA328.PD3(INT1), R9.1, RTC.INT/SQW
- new net SCL: R2.1, SIGNAL_ISOLATOR.I/OA2, TO_MASTER_BOARD.4
- new net SCL_ISO: ATMEGA328.PC5(ADC5/SCL), R5.1, SIGNAL_ISOLATOR.I/OB2
- new net SDA: R3.1, SIGNAL_ISOLATOR.I/OA1, TO_MASTER_BOARD.3
- new net SDA_ISO: ATMEGA328.PC4(ADC4/SDA), R4.1, SIGNAL_ISOLATOR.I/OB1
- new net VREF_2V5: 2V5_VOLTAGE_REF.VOUT_FORCE, 2V5_VOLTAGE_REF.VOUT_SEN, ADC.VREFP, C16.1, C3.1, C4.1, C5.1
- net AIN0: now also ADC.AIN0; no longer U1.AIN0
- net AIN1: now also ADC.AIN1; no longer U1.AIN1
- net AIN2: now also ADC.AIN2; no longer U1.AIN2
- net AIN3: now also ADC.AIN3; no longer U1.AIN3
- net AIN4: now also ADC.AIN4; no longer U1.AIN4
- net AIN5: now also ADC.AIN5; no longer U1.AIN5
- net N$11: now also ADC.XTAL1/CLKIN; no longer U1.XTAL1/CLKIN
- net N$12: now also ADC.XTAL2; no longer U1.XTAL2
- net N$13: now also ATMEGA328.PB6(XTAL1/TOSC1), C32.2, Q2.1; no longer DIG_OUT.3, U1.D2
- net N$16: now also ADC.~CS, R8.1; no longer R7.1, SERIAL.2
- net N$17: now also ADC.~RESET, SJ1.2; no longer R6.1, SERIAL.1
- net N$18: now also ADC.AIN6; no longer U1.AIN6
- net N$19: now also ADC.AIN7; no longer U1.AIN7
- net N$6: now also ATMEGA328.PB7(XTAL2/TOSC2), C33.2, Q2.2; no longer DIG_OUT.2, U1.D1
- net SCLK: now also ATMEGA328.PB5(SCK), ICSP.3, RTC.SCLK@18, RTC.SCLK@20; no longer U1.SCLK
Other:
- note added: "3V3 Regulator"
- note added: "Analog-Digital Conversion"
- note removed: "DS1256 ADC"
- moved on the sheet: AIN6-7, ATMEGA328, C1, C10, C11, C12, C13, C14, C15, C16, C17, C2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

Commit message: Almost finished the first version. I have to finish the current path and check everything
Parts:
- added JP1: (no value), adafruit:PINHD-1X3
Connections:
- net 1WIRE_BUS: now also JP1.2
- net 5V_ISO: now also JP1.1; no longer C27.2, SIGNAL_ISOLATOR.GNDB
- net GND_ISO: now also C27.2, JP1.3, SIGNAL_ISOLATOR.GNDB
- net IN2_ISO: now also ATMEGA328.PD5(T1)
- net OUT2_ISO: now also ATMEGA328.PB2(SS/OC1B)
Other:
- moved on the sheet: ICSP, TO_MASTER_BOARD
Changed lines of the file:
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@@
 <part name="R10" library="SparkFun-Passives" deviceset="RESISTOR" device="1206" value="4.7k"/>
 <part name="R11" library="SparkFun-Passives" deviceset="RESISTOR" device="1206" value="10k"/>
+<part name="JP1" library="adafruit" deviceset="PINHD-1X3" device=""/>
 </parts>
 <sheets>
@@
 <instance part="ATMEGA328" gate="U$1" x="109.22" y="-223.52"/>
 <instance part="RTC" gate="G$1" x="50.8" y="-78.74"/>
-<instance part="ICSP" gate="G$1" x="365.76" y="-182.88"/>
+<instance part="ICSP" gate="G$1" x="408.94" y="-175.26"/>
 <instance part="RESET_BUTTON" gate="S" x="71.12" y="-177.8"/>
 <instance part="DC-DC" gate="A" x="396.24" y="86.36"/>
 <instance part="SIGNAL_ISOLATOR" gate="IC" x="396.24" y="20.32"/>
-<instance part="TO_MASTER_BOARD" gate="A" x="457.2" y="-177.8"/>
+<instance part="TO_MASTER_BOARD" gate="A" x="480.06" y="-177.8"/>
 <instance part="C18" gate="G$1" x="345.44" y="88.9"/>
 <instance part="C19" gate="G$1" x="353.06" y="88.9"/>
@@
 <instance part="R10" gate="G$1" x="180.34" y="-218.44" rot="R270"/>
 <instance part="R11" gate="G$1" x="68.58" y="-193.04"/>
+<instance part="JP1" gate="A" x="353.06" y="-180.34"/>
 </instances>
 <busses>
@@
 <segment>
 <pinref part="ICSP" gate="G$1" pin="3"/>
-<wire x1="358.14" y1="-182.88" x2="345.44" y2="-182.88" width="0.1524" layer="91"/>
-<label x="345.44" y="-182.88" size="1.778" layer="95" rot="R180" xref="yes"/>
+<wire x1="401.32" y1="-175.26" x2="388.62" y2="-175.26" width="0.1524" layer="91"/>
+<label x="388.62" y="-175.26" size="1.778" layer="95" rot="R180" xref="yes"/>
 </segment>
 </net>
@@
 <segment>
 <pinref part="TO_MASTER_BOARD" gate="A" pin="1"/>
-<wire x1="454.66" y1="-167.64" x2="439.42" y2="-167.64" width="0.1524" layer="91"/>
-<label x="439.42" y="-167.64" size="1.778" layer="95" rot="R180" xref="yes"/>
+<wire x1="477.52" y1="-167.64" x2="462.28" y2="-167.64" width="0.1524" layer="91"/>
+<label x="462.28" y="-167.64" size="1.778" layer="95" rot="R180" xref="yes"/>
 </segment>
 <segment>
@@
 <segment>
 <pinref part="ICSP" gate="G$1" pin="2"/>
-<wire x1="373.38" y1="-180.34" x2="375.92" y2="-180.34" width="0.1524" layer="91"/>
-<label x="375.92" y="-180.34" size="1.778" layer="95" xref="yes"/>
+<wire x1="416.56" y1="-172.72" x2="419.1" y2="-172.72" width="0.1524" layer="91"/>
+<label x="419.1" y="-172.72" size="1.778" layer="95" xref="yes"/>
 </segment>
 </net>
@@
 <segment>
 <pinref part="TO_MASTER_BOARD" gate="A" pin="2"/>
-<wire x1="454.66" y1="-170.18" x2="447.04" y2="-170.18" width="0.1524" layer="91"/>
-<label x="447.04" y="-170.18" size="1.778" layer="95" rot="R180" xref="yes"/>
+<wire x1="477.52" y1="-170.18" x2="469.9" y2="-170.18" width="0.1524" layer="91"/>
+<label x="469.9" y="-170.18" size="1.778" layer="95" rot="R180" xref="yes"/>
 </segment>
 <segment>
@@
 <segment>
 <pinref part="ICSP" gate="G$1" pin="6"/>
-<wire x1="373.38" y1="-185.42" x2="375.92" y2="-185.42" width="0.1524" layer="91"/>
-<label x="375.92" y="-185.42" size="1.778" layer="95" xref="yes"/>
+<wire x1="416.56" y1="-177.8" x2="419.1" y2="-177.8" width="0.1524" layer="91"/>
+<label x="419.1" y="-177.8" size="1.778" layer="95" xref="yes"/>
 </segment>
 </net>
@@
 <segment>
 <pinref part="TO_MASTER_BOARD" gate="A" pin="3"/>
-<wire x1="454.66" y1="-172.72" x2="439.42" y2="-172.72" width="0.1524" layer="91"/>
-<label x="439.42" y="-172.72" size="1.778" layer="95" rot="R180" xref="yes"/>
+<wire x1="477.52" y1="-172.72" x2="462.28" y2="-172.72" width="0.1524" layer="91"/>
+<label x="462.28" y="-172.72" size="1.778" layer="95" rot="R180" xref="yes"/>
 </segment>
 <segment>
@@
 <segment>
 <pinref part="TO_MASTER_BOARD" gate="A" pin="4"/>
-<wire x1="454.66" y1="-175.26" x2="447.04" y2="-175.26" width="0.1524" layer="91"/>
-<label x="447.04" y="-175.26" size="1.778" layer="95" rot="R180" xref="yes"/>
+<wire x1="477.52" y1="-175.26" x2="469.9" y2="-175.26" width="0.1524" layer="91"/>
+<label x="469.9" y="-175.26" size="1.778" layer="95" rot="R180" xref="yes"/>
 </segment>
 <segment>
@@
 <wire x1="457.2" y1="25.4" x2="457.2" y2="27.94" width="0.1524" layer="91"/>
 <junction x="457.2" y="27.94"/>
-</segment>
-<segment>
-<pinref part="SIGNAL_ISOLATOR" gate="IC" pin="GNDB"/>
-<wire x1="403.86" y1="10.16" x2="474.98" y2="10.16" width="0.1524" layer="91"/>
-<pinref part="C27" gate="G$1" pin="2"/>
-<wire x1="474.98" y1="10.16" x2="480.06" y2="10.16" width="0.1524" layer="91"/>
-<wire x1="474.98" y1="15.24" x2="474.98" y2="10.16" width="0.1524" layer="91"/>
-<junction x="474.98" y="10.16"/>
-<label x="480.06" y="10.16" size="1.778" layer="95" xref="yes"/>
 </segment>
 <segment>
@@
 <wire x1="180.34" y1="-210.82" x2="187.96" y2="-210.82" width="0.1524" layer="91"/>
 <label x="187.96" y="-210.82" size="1.778" layer="95" xref="yes"/>
+</segment>
+<segment>
+<pinref part="JP1" gate="A" pin="1"/>
+<wire x1="350.52" y1="-177.8" x2="342.9" y2="-177.8" width="0.1524" layer="91"/>
+<label x="342.9" y="-177.8" size="1.778" layer="95" rot="R180" xref="yes"/>
 </segment>
 </net>
@@
 <label x="58.42" y="-177.8" size="1.778" layer="95" rot="R180" xref="yes"/>
 </segment>
+<segment>
+<pinref part="SIGNAL_ISOLATOR" gate="IC" pin="GNDB"/>
+<wire x1="403.86" y1="10.16" x2="474.98" y2="10.16" width="0.1524" layer="91"/>
+<pinref part="C27" gate="G$1" pin="2"/>
+<wire x1="474.98" y1="10.16" x2="480.06" y2="10.16" width="0.1524" layer="91"/>
+<wire x1="474.98" y1="15.24" x2="474.98" y2="10.16" width="0.1524" layer="91"/>
+<junction x="474.98" y="10.16"/>
+<label x="480.06" y="10.16" size="1.778" layer="95" xref="yes"/>
+</segment>
+<segment>
+<pinref part="JP1" gate="A" pin="3"/>
+<wire x1="350.52" y1="-182.88" x2="345.44" y2="-182.88" width="0.1524" layer="91"/>
+<label x="345.44" y="-182.88" size="1.778" layer="95" rot="R180" xref="yes"/>
+</segment>
 </net>
 <net name="IN2_ISO" class="0">
@@
 <label x="426.72" y="22.86" size="1.778" layer="95" xref="yes"/>
 </segment>
+<segment>
+<pinref part="ATMEGA328" gate="U$1" pin="PD5(T1)"/>
+<wire x1="132.08" y1="-228.6" x2="134.62" y2="-228.6" width="0.1524" layer="91"/>
+<label x="134.62" y="-228.6" size="1.778" layer="95" xref="yes"/>
+</segment>
 </net>
 <net name="OUT1_ISO" class="0">
@@
 <wire x1="403.86" y1="17.78" x2="426.72" y2="17.78" width="0.1524" layer="91"/>
 <label x="426.72" y="17.78" size="1.778" layer="95" xref="yes"/>
+</segment>
+<segment>
+<pinref part="ATMEGA328" gate="U$1" pin="PB2(SS/OC1B)"/>
+<wire x1="132.08" y1="-243.84" x2="165.1" y2="-243.84" width="0.1524" layer="91"/>
+<label x="165.1" y="-243.84" size="1.778" layer="95" xref="yes"/>
 </segment>
 </net>
@@
 <segment>
 <pinref part="TO_MASTER_BOARD" gate="A" pin="6"/>
-<wire x1="454.66" y1="-180.34" x2="447.04" y2="-180.34" width="0.1524" layer="91"/>
-<label x="447.04" y="-180.34" size="1.778" layer="95" rot="R180" xref="yes"/>
+<wire x1="477.52" y1="-180.34" x2="469.9" y2="-180.34" width="0.1524" layer="91"/>
+<label x="469.9" y="-180.34" size="1.778" layer="95" rot="R180" xref="yes"/>
 </segment>
 </net>
@@
 <segment>
 <pinref part="TO_MASTER_BOARD" gate="A" pin="5"/>
-<wire x1="454.66" y1="-177.8" x2="439.42" y2="-177.8" width="0.1524" layer="91"/>
-<label x="439.42" y="-177.8" size="1.778" layer="95" rot="R180" xref="yes"/>
+<wire x1="477.52" y1="-177.8" x2="462.28" y2="-177.8" width="0.1524" layer="91"/>
+<label x="462.28" y="-177.8" size="1.778" layer="95" rot="R180" xref="yes"/>
 </segment>
 </net>
@@
 <segment>
 <pinref part="TO_MASTER_BOARD" gate="A" pin="7"/>
-<wire x1="454.66" y1="-182.88" x2="436.88" y2="-182.88" width="0.1524" layer="91"/>
-<label x="436.88" y="-182.88" size="1.778" layer="95" rot="R180" xref="yes"/>
+<wire x1="477.52" y1="-182.88" x2="459.74" y2="-182.88" width="0.1524" layer="91"/>
+<label x="459.74" y="-182.88" size="1.778" layer="95" rot="R180" xref="yes"/>
 </segment>
 </net>
@@
 <segment>
 <pinref part="TO_MASTER_BOARD" gate="A" pin="8"/>
-<wire x1="454.66" y1="-185.42" x2="447.04" y2="-185.42" width="0.1524" layer="91"/>
-<label x="447.04" y="-185.42" size="1.778" layer="95" rot="R180" xref="yes"/>
+<wire x1="477.52" y1="-185.42" x2="469.9" y2="-185.42" width="0.1524" layer="91"/>
+<label x="469.9" y="-185.42" size="1.778" layer="95" rot="R180" xref="yes"/>
 </segment>
 </net>
@@
 <segment>
 <pinref part="ICSP" gate="G$1" pin="1"/>
-<wire x1="358.14" y1="-180.34" x2="355.6" y2="-180.34" width="0.1524" layer="91"/>
-<label x="355.6" y="-180.34" size="1.778" layer="95" rot="R180" xref="yes"/>
+<wire x1="401.32" y1="-172.72" x2="398.78" y2="-172.72" width="0.1524" layer="91"/>
+<label x="398.78" y="-172.72" size="1.778" layer="95" rot="R180" xref="yes"/>
 </segment>
 </net>
@@
 <segment>
 <pinref part="ICSP" gate="G$1" pin="4"/>
-<wire x1="373.38" y1="-182.88" x2="383.54" y2="-182.88" width="0.1524" layer="91"/>
-<label x="383.54" y="-182.88" size="1.778" layer="95" xref="yes"/>
+<wire x1="416.56" y1="-175.26" x2="426.72" y2="-175.26" width="0.1524" layer="91"/>
+<label x="426.72" y="-175.26" size="1.778" layer="95" xref="yes"/>
 </segment>
 </net>
@@
 <wire x1="180.34" y1="-223.52" x2="180.34" y2="-226.06" width="0.1524" layer="91"/>
 <junction x="180.34" y="-226.06"/>
+</segment>
+<segment>
+<pinref part="JP1" gate="A" pin="2"/>
+<wire x1="350.52" y1="-180.34" x2="330.2" y2="-180.34" width="0.1524" layer="91"/>
+<label x="330.2" y="-180.34" size="1.778" layer="95" rot="R180" xref="yes"/>
 </segment>
 </net>
@@
 <segment>
 <pinref part="ICSP" gate="G$1" pin="5"/>
-<wire x1="358.14" y1="-185.42" x2="355.6" y2="-185.42" width="0.1524" layer="91"/>
-<label x="355.6" y="-185.42" size="1.778" layer="95" rot="R180" xref="yes"/>
-</segment>
-</net>
+<wire x1="401.32" y1="-177.8" x2="398.78" y2="-177.8" width="0.1524" layer="91"/>
+<label x="398.78" y="-177.8" size="1.778" layer="95" rot="R180" xref="yes"/>
+</segment>
+</net>

Commit message: finished the first draft version of the board
Other:
- note added: "This board measures Voltage, Current and Temperature of a PV panel.In addition, it gets Date and Time stamp. The data are collected by the microprocessor Atmega328 and send out as I2C packages to master board. Every connection outside the board is isolated. (NOMINAL 40V@8A, MAX 45V@15A)"
- note removed: "This board measures Voltage, Current and Temperature. In addition, it get a Date and Time stamp. The data are collected from the microprocessor Atmega328 and send out as I2C packages. Isolation is placed in every connection outside the board"
- moved on the sheet: 2V5_VOLTAGE_REF, 3V3_REGULATOR, ADC, AIN6-7, ATMEGA328, C1, C10, C11, C12, C13, C14, C15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
