File: board1.brd (EAGLE design)
At the start: 100 x 80 mm, 73 parts, among them Q1 7.68M, Q2 16MHz

Commit message: Started wiring for the first DRAFT version
Parts:
- moved R3 24.4 mm to (17.8, 11.4), turned to 90 degrees
- moved R2 23.3 mm to (17.8, 16.5), turned to 270 degrees
- moved C27 6.35 mm to (31.8, 33.0), turned to 270 degrees
- moved C26 4.58 mm to (19.1, 33.0)
- moved SIGNAL_ISOLATOR 1.80 mm to (25.4, 24.1), turned to 270 degrees
- moved C22 1.27 mm to (49.5, 14.0), turned to 270 degrees
- moved C23 1.27 mm to (53.3, 14.0), turned to 270 degrees
- moved C20 1.27 mm to (25.4, 6.35), turned to 270 degrees
- moved C21 1.27 mm to (29.2, 6.35), turned to 270 degrees
Routing:
- net GND: track 0.00 -> 121.4 mm, vias 0 -> 4
- net 5V: track 0.00 -> 117.9 mm, vias 0 -> 4
- net 5V_ISO: track 0.00 -> 74.3 mm, vias 0 -> 2
- net VBUS1: track 0.00 -> 56.8 mm
- net GND_ISO: track 0.00 -> 34.5 mm, vias 0 -> 2
- net IN1: track 0.00 -> 34.3 mm
- net SDA: track 0.00 -> 34.0 mm, vias 0 -> 2
- net IN2: track 0.00 -> 27.9 mm
- net OUT1: track 0.00 -> 21.6 mm
- net VBUS2: track 0.00 -> 20.7 mm
- net AIN3: track 0.00 -> 18.2 mm
- net SCL: track 0.00 -> 16.8 mm
- net AIN5: track 0.00 -> 13.6 mm
- net OUT2: track 0.00 -> 10.9 mm
- net N$9: track 0.00 -> 3.68 mm
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
Commit message: Almost finished the first version. I have to finish the current path and check everything
Parts:
- added JP1: (no value), adafruit:1X03
- moved R8 50.3 mm to (34.9, 50.2), turned to 180 degrees
- moved C33 21.1 mm to (21.0, 62.2)
- moved C34 18.8 mm to (24.1, 38.7), turned to 180 degrees
- moved C32 16.2 mm to (23.5, 62.2), turned to 270 degrees
- moved R6 16.1 mm to (76.2, 26.7), turned to 90 degrees
- moved Q2 11.4 mm to (22.2, 55.9), turned to 180 degrees
- moved R9 8.35 mm to (34.9, 53.3), turned to 0 degrees
- moved R10 7.65 mm to (13.3, 67.3)
- moved ATMEGA328 7.24 mm to (24.8, 46.4), turned to 270 degrees
- moved C16 5.08 mm to (91.4, 44.5)
- moved 2V5_VOLTAGE_REF 5.08 mm to (91.4, 39.4)
- moved C17 5.08 mm to (91.4, 34.3), turned to 180 degrees
- moved R7 4.58 mm to (81.3, 26.7), turned to 90 degrees
- moved AIN6-7 3.86 mm to (50.8, 42.5), turned to 90 degrees
- moved C31 3.59 mm to (78.7, 14.0), turned to 0 degrees
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Connections:
- net 1WIRE_BUS: now also JP1.2
- net 5V_ISO: now also JP1.1; no longer C27.2, SIGNAL_ISOLATOR.9
- net GND_ISO: now also C27.2, JP1.3, SIGNAL_ISOLATOR.9
- net IN2_ISO: now also ATMEGA328.9
- net OUT2_ISO: now also ATMEGA328.14
Routing:
- net GND_ISO: track 34.5 -> 565.0 mm, vias 2 -> 13
- net SCLK: track 0.00 -> 229.4 mm, vias 0 -> 7
- net 5V_ISO: track 74.3 -> 293.8 mm, vias 2 -> 6
- net MISO: track 0.00 -> 193.3 mm, vias 0 -> 4
- net MOSI: track 0.00 -> 131.6 mm, vias 0 -> 7
- net RTC_SQW: track 0.00 -> 120.2 mm, vias 0 -> 2
- net 3V3: track 0.00 -> 114.2 mm, vias 0 -> 2
- net RTC_CS: track 0.00 -> 111.4 mm, vias 0 -> 2
- net VREF_2V5: track 0.00 -> 102.8 mm
- net RESET: track 0.00 -> 69.3 mm, vias 0 -> 3
- net SCL_ISO: track 0.00 -> 58.2 mm, vias 0 -> 2
- net AIN5: track 13.6 -> 71.6 mm, vias 0 -> 2
- net ADC_DRDY: track 0.00 -> 54.7 mm, vias 0 -> 4
- net OUT2_ISO: track 0.00 -> 50.3 mm, vias 0 -> 2
- net N$16: track 0.00 -> 50.2 mm, vias 0 -> 2
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- added copper zone on layer 1, net N$15
- added copper zone on layer 1, net N$22
- added copper zone on layer 1, net N$23
- added copper zone on layer 1, net N$24

Commit message: finished the first draft version of the board
Routing:
- net VBUS1: track 17.0 -> 50.6 mm
- net GND_ISO: track 565.0 -> 567.5 mm
- added copper zone on layer 1, net AIN3
- added copper zone on layer 1, net AIN5
- added copper zone on layer 1, net VBUS1
- added copper zone on layer 1, net VBUS2
- removed copper zone on layer 1, net N$15
- removed copper zone on layer 1, net N$22
- removed copper zone on layer 1, net N$23
- removed copper zone on layer 1, net N$24
Other:
- board text added: "Measuring PCB v1.0"
Changed lines of the file:
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@@
 <wire x1="100" y1="80" x2="0" y2="80" width="0" layer="20"/>
 <wire x1="0" y1="80" x2="0" y2="0" width="0" layer="20"/>
+<text x="1.905" y="76.835" size="1.778" layer="1">Measuring PCB v1.0</text>
 </plain>
 <attributes>
@@
 <contactref element="JP1B" pad="2"/>
 <wire x1="34.29" y1="74.93" x2="34.29" y2="76.2" width="1.016" layer="1"/>
-<wire x1="34.29" y1="76.2" x2="35.56" y2="77.47" width="1.016" layer="1"/>
-<wire x1="35.56" y1="77.47" x2="46.99" y2="77.47" width="1.016" layer="1"/>
-<wire x1="46.99" y1="74.93" x2="46.99" y2="77.47" width="1.016" layer="1"/>
-<wire x1="77.39" y1="73.66" x2="85.17" y2="73.66" width="0" layer="19" extent="1-1"/>
-<wire x1="46.99" y1="74.93" x2="77.39" y2="73.66" width="0" layer="19" extent="1-1"/>
+<wire x1="34.29" y1="76.2" x2="36.195" y2="78.105" width="1.016" layer="1"/>
+<wire x1="36.195" y1="78.105" x2="46.99" y2="78.105" width="1.016" layer="1"/>
+<wire x1="46.99" y1="74.93" x2="46.99" y2="78.105" width="1.016" layer="1"/>
+<polygon width="0.4064" layer="1" thermals="no">
+<vertex x="88.265" y="73.66"/>
+<vertex x="88.265" y="71.12"/>
+<vertex x="86.36" y="69.215"/>
+<vertex x="76.2" y="69.215"/>
+<vertex x="74.295" y="71.12"/>
+<vertex x="74.295" y="75.565"/>
+<vertex x="76.2" y="77.47"/>
+<vertex x="86.36" y="77.47"/>
+<vertex x="88.265" y="75.565"/>
+</polygon>
+<wire x1="46.99" y1="78.105" x2="73.66" y2="78.105" width="1.016" layer="1"/>
+<wire x1="73.66" y1="78.105" x2="76.835" y2="74.93" width="1.016" layer="1"/>
+<wire x1="76.835" y1="74.93" x2="76.835" y2="74.215" width="1.016" layer="1"/>
+<wire x1="76.835" y1="74.215" x2="77.39" y2="73.66" width="1.016" layer="1"/>
 </signal>
 <signal name="N$2">
@@
 <wire x1="52.705" y1="55.88" x2="61.595" y2="64.77" width="0.6096" layer="16"/>
 <via x="61.595" y="64.77" extent="1-16" drill="0.6"/>
-<wire x1="61.595" y1="64.77" x2="67.39" y2="73.66" width="0" layer="19" extent="1-1"/>
-<wire x1="64.24" y1="59.3" x2="61.595" y2="64.77" width="0" layer="19" extent="1-1"/>
+<polygon width="0.4064" layer="1" thermals="no">
+<vertex x="65.405" y="76.2"/>
+<vertex x="69.215" y="76.2"/>
+<vertex x="70.485" y="75.565"/>
+<vertex x="70.485" y="71.12"/>
+<vertex x="64.77" y="64.77"/>
+<vertex x="64.77" y="58.42"/>
+<vertex x="61.595" y="58.42"/>
+<vertex x="59.69" y="60.325"/>
+<vertex x="59.69" y="70.485"/>
+</polygon>
 </signal>
 <signal name="AIN5">
@@
 <wire x1="63.5" y1="62.865" x2="71.12" y2="62.865" width="0.6096" layer="16"/>
 <via x="71.12" y="62.865" extent="1-16" drill="0.6"/>
-<wire x1="74.676" y1="61.595" x2="79.756" y2="61.595" width="0" layer="19" extent="1-1"/>
-<wire x1="71.12" y1="62.865" x2="74.676" y2="61.595" width="0" layer="19" extent="1-1"/>
-<wire x1="67.84" y1="59.3" x2="71.12" y2="62.865" width="0" layer="19" extent="1-1"/>
+<polygon width="0.4064" layer="1" thermals="no">
+<vertex x="67.945" y="58.42"/>
+<vertex x="81.28" y="58.42"/>
+<vertex x="83.185" y="60.325"/>
+<vertex x="83.185" y="63.5"/>
+<vertex x="80.645" y="66.04"/>
+<vertex x="69.85" y="66.04"/>
+<vertex x="67.945" y="64.135"/>
+</polygon>
 </signal>
 <signal name="VBUS2">
@@
 <contactref element="VPANEL" pad="2"/>
 <contactref element="F1" pad="1B"/>
-<wire x1="95.504" y1="61.595" x2="95.17" y2="73.66" width="0" layer="19" extent="1-1"/>
-<wire x1="90.424" y1="61.595" x2="95.504" y2="61.595" width="0" layer="19" extent="1-1"/>
+<polygon width="0.4064" layer="1" thermals="no">
+<vertex x="92.075" y="76.835"/>
+<vertex x="96.52" y="76.835"/>
+<vertex x="98.425" y="74.93"/>
+<vertex x="98.425" y="59.055"/>
+<vertex x="96.52" y="57.15"/>
+<vertex x="90.17" y="57.15"/>
+<vertex x="87.63" y="59.69"/>
+<vertex x="87.63" y="67.31"/>
+<vertex x="90.805" y="70.485"/>
+<vertex x="90.805" y="75.565"/>
+</polygon>
 </signal>
 <signal name="AIN1">
@@
 <wire x1="27.81" y1="63.63" x2="29.21" y2="62.23" width="0.6096" layer="1"/>
 <via x="29.21" y="62.23" extent="1-16" drill="0.6"/>
-<wire x1="29.21" y1="62.23" x2="31.75" y2="59.69" width="0.6096" layer="16"/>
-<wire x1="31.75" y1="59.69" x2="39.37" y2="59.69" width="0.6096" layer="16"/>
-<wire x1="39.37" y1="59.69" x2="41.91" y2="57.15" width="0.6096" layer="16"/>
-<wire x1="41.91" y1="57.15" x2="41.91" y2="38.735" width="0.6096" layer="16"/>
 <wire x1="41.91" y1="38.735" x2="34.925" y2="31.75" width="0.6096" layer="16"/>
 <wire x1="71.0946" y1="7.62" x2="66.675" y2="7.62" width="0.4064" layer="1"/>
@@
 <wire x1="30.48" y1="17.78" x2="48.26" y2="17.78" width="0.4064" layer="16"/>
 <wire x1="48.26" y1="17.78" x2="55.88" y2="10.16" width="0.4064" layer="16"/>
-<wire x1="51.435" y1="24.635" x2="53.845" y2="24.635" width="0.4064" layer="1"/>
-<wire x1="53.845" y1="24.635" x2="53.975" y2="24.765" width="0.4064" layer="1"/>
-<wire x1="53.975" y1="24.765" x2="64.135" y2="24.765" width="0.4064" layer="1"/>
-<wire x1="64.389" y1="26.8478" x2="64.389" y2="25.019" width="0.4064" layer="1"/>
-<wire x1="64.389" y1="25.019" x2="64.135" y2="24.765" width="0.4064" layer="1"/>
 <wire x1="51.435" y1="24.635" x2="49.025" y2="24.635" width="0.4064" layer="1"/>
 <wire x1="49.025" y1="24.635" x2="41.91" y2="31.75" width="0.4064" layer="1"/>
@@
 <wire x1="90.805" y1="15.875" x2="91.44" y2="16.51" width="0.4064" layer="1"/>
 <wire x1="91.44" y1="16.51" x2="92.075" y2="16.51" width="0.4064" layer="1"/>
-<wire x1="53.975" y1="24.765" x2="54.61" y2="24.635" width="0" layer="19" extent="1-1"/>
-<wire x1="64.77" y1="6.855" x2="63.5" y2="6.35" width="0" layer="19" extent="1-16"/>
+<wire x1="29.21" y1="62.23" x2="41.91" y2="49.53" width="0.6096" layer="16"/>
+<wire x1="41.91" y1="49.53" x2="41.91" y2="38.735" width="0.6096" layer="16"/>
+<wire x1="64.77" y1="6.855" x2="58.925" y2="6.855" width="0.4064" layer="1"/>
+<wire x1="58.925" y1="6.855" x2="58.42" y2="6.35" width="0.4064" layer="1"/>
+<wire x1="64.389" y1="26.8478" x2="64.389" y2="25.019" width="0.4064" layer="1"/>
+<wire x1="64.389" y1="25.019" x2="63.5" y2="24.13" width="0.4064" layer="1"/>
+<wire x1="63.5" y1="24.13" x2="55.115" y2="24.13" width="0.4064" layer="1"/>
+<wire x1="55.115" y1="24.13" x2="54.61" y2="24.635" width="0.4064" layer="1"/>
+<wire x1="54.61" y1="24.635" x2="51.435" y2="24.635" width="0.4064" layer="1"/>
 </signal>
 <signal name="IN2_ISO">
@@
 <wire x1="26.67" y1="34.925" x2="26.67" y2="44.45" width="0.4064" layer="16"/>
 </signal>
-<signal name="N$15">
-<polygon width="0.4064" layer="1">
-<vertex x="92.075" y="76.835"/>
-<vertex x="96.52" y="76.835"/>
-<vertex x="98.425" y="74.93"/>
-<vertex x="98.425" y="59.055"/>
-<vertex x="96.52" y="57.15"/>
-<vertex x="90.17" y="57.15"/>
-<vertex x="87.63" y="59.69"/>
-<vertex x="87.63" y="67.31"/>
-<vertex x="90.805" y="70.485"/>
-<vertex x="90.805" y="75.565"/>
-</polygon>
-</signal>
-<signal name="N$22">
-<polygon width="0.4064" layer="1">
-<vertex x="88.265" y="73.66"/>
-<vertex x="88.265" y="71.12"/>
-<vertex x="86.36" y="69.215"/>
-<vertex x="76.2" y="69.215"/>
-<vertex x="74.295" y="71.12"/>
-<vertex x="74.295" y="75.565"/>
-<vertex x="76.2" y="77.47"/>
-<vertex x="86.36" y="77.47"/>
-<vertex x="88.265" y="75.565"/>
-</polygon>
-</signal>
-<signal name="N$23">
-<polygon width="0.4064" layer="1">
-<vertex x="67.945" y="58.42"/>
-<vertex x="81.28" y="58.42"/>
-<vertex x="83.185" y="60.325"/>
-<vertex x="83.185" y="63.5"/>
-<vertex x="80.645" y="66.04"/>
-<vertex x="69.85" y="66.04"/>
-<vertex x="67.945" y="64.135"/>
-</polygon>
-</signal>
-<signal name="N$24">
-<polygon width="0.4064" layer="1">
-<vertex x="66.04" y="76.835"/>
-<vertex x="69.85" y="76.835"/>
-<vertex x="71.12" y="75.565"/>
-<vertex x="71.12" y="71.12"/>
-<vertex x="64.77" y="64.77"/>
-<vertex x="64.77" y="58.42"/>
-<vertex x="61.595" y="58.42"/>
-<vertex x="59.69" y="60.325"/>
-<vertex x="59.69" y="70.485"/>
-</polygon>
-</signal>
 </signals>
